File: hardware/kicad/elderly-companion-robot/audio.kicad_sch (KiCad schematic)
At the start: 0 parts

Commit message: Phase 9-10: All 6 hierarchical sheets populated with components, labels, and power symbols
- Power_Supply: LM2596S-5 buck, AP2112K-3.3 LDO, AMS1117-ADJ (4V for SIM800L),
  TP4056 charger, caps, diodes, connectors, resistor dividers
- MCU_Core: ESP32-S3-WROOM-1, 8x decoupling caps, boot/EN resistors,
  hierarchical labels for all peripheral interfaces
- Motor_Driver: L298N, 8x flyback diodes, motor connectors, hierarchical labels
- Sensors: MPU-6050, SSD1306 OLED, 4x HC-SR04 connectors, voltage dividers,
  I2C pull-ups, hierarchical labels
- Audio: MAX98357A, INMP441 connector (6-pin), speaker connector, bypass caps,
  I2S hierarchical labels
- Camera_Dock: SIM800C, 2x servo connectors, IR TX/RX, dock contact,
  UART2/PWRKEY hierarchical labels
- Top-level schematic restored with 6 hierarchical sheet references
- ERC: 0 violations
- Quality gate: Schematic PASS

Co-Authored-By: Claude Opus 4.7 <noreply@anthropic.com>
Parts:
- added C31, C33: 100nF, Capacitor_SMD:C_0402_1005Metric, symbol Device:C
- added C32: 10uF, Capacitor_SMD:C_0805_2012Metric, symbol Device:C
- added J10: Speaker, Connector_PinHeader_2.54mm:PinHeader_1x02_P2.54mm_Vertical, symbol Connector_Generic:Conn_01x02
- added J9: INMP441_Mic, Connector_PinHeader_2.54mm:PinHeader_1x06_P2.54mm_Vertical, symbol Connector_Generic:Conn_01x06
- added R17: 10K, Resistor_SMD:R_0402_1005Metric, symbol Device:R
- added U8: MAX98357A, Package_QFP:TQFP-16_3x3mm_P0.5mm, symbol Audio:MAX98357A
Connections:
- new net: U8.11 (GND), U8.15 (GND), U8.3 (GND)
- new net: U8.7 (VDD), U8.8 (VDD)
Other:
- title: Audio -> (none)

Commit message: LCSC part binding + all 6 sheets wired, ERC clean
- LCSC codes bound for passive components (caps, resistors, diodes, LEDs)
- Power Supply: LM2596S-5, AP2112K, AMS1117, TP4056 wired with nets
- MCU Core: ESP32-S3-WROOM-1 + decoupling caps + hierarchical labels
- Motor Driver: L298N + flyback diodes + connectors + labels
- Sensors: MPU-6050, SSD1306, 4x HC-SR04 + voltage dividers
- Audio: MAX98357A, INMP441 connector, speaker + I2S labels
- Camera/Dock: SIM800C, servos, IR, dock contact + UART2 labels
- ERC: 0 violations, schematic quality gate PASS

Co-Authored-By: Claude Opus 4.7 <noreply@anthropic.com>
Parts:
- C31, C33: footprint Capacitor_SMD:C_0402_1005Metric -> 0402; LCSC (none) -> C1525; MPN (none) -> CL05B104KO5NNNC
- C32: footprint Capacitor_SMD:C_0805_2012Metric -> 0805; LCSC (none) -> C15850; MPN (none) -> CL21A106KAYNNNE
- R17: footprint Resistor_SMD:R_0402_1005Metric -> 0402; LCSC (none) -> C25744; MPN (none) -> 0402WGF1002TCE
Changed lines of the file:
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@@
 			(effects (font (size 1.27 1.27)))
 		)
-		(property "Footprint" "Capacitor_SMD:C_0402_1005Metric"
+		(property "Footprint" "0402"
 			(at 127 50.8 0)
 			(effects (font (size 1.27 1.27)) (hide yes))
 		)
 		(property "Datasheet" "~"
+			(at 127 50.8 0)
+			(effects (font (size 1.27 1.27)) (hide yes))
+		)
+		(property "LCSC" "C1525"
+			(at 127 50.8 0)
+			(effects (font (size 1.27 1.27)) (hide yes))
+		)
+		(property "MPN" "CL05B104KO5NNNC"
 			(at 127 50.8 0)
 			(effects (font (size 1.27 1.27)) (hide yes))
@@
 			(effects (font (size 1.27 1.27)))
 		)
-		(property "Footprint" "Capacitor_SMD:C_0805_2012Metric"
+		(property "Footprint" "0805"
 			(at 152.4 50.8 0)
 			(effects (font (size 1.27 1.27)) (hide yes))
 		)
 		(property "Datasheet" "~"
+			(at 152.4 50.8 0)
+			(effects (font (size 1.27 1.27)) (hide yes))
+		)
+		(property "LCSC" "C15850"
+			(at 152.4 50.8 0)
+			(effects (font (size 1.27 1.27)) (hide yes))
+		)
+		(property "MPN" "CL21A106KAYNNNE"
 			(at 152.4 50.8 0)
 			(effects (font (size 1.27 1.27)) (hide yes))
@@
 			(effects (font (size 1.27 1.27)))
 		)
-		(property "Footprint" "Capacitor_SMD:C_0402_1005Metric"
+		(property "Footprint" "0402"
 			(at 177.8 50.8 0)
 			(effects (font (size 1.27 1.27)) (hide yes))
 		)
 		(property "Datasheet" "~"
+			(at 177.8 50.8 0)
+			(effects (font (size 1.27 1.27)) (hide yes))
+		)
+		(property "LCSC" "C1525"
+			(at 177.8 50.8 0)
+			(effects (font (size 1.27 1.27)) (hide yes))
+		)
+		(property "MPN" "CL05B104KO5NNNC"
 			(at 177.8 50.8 0)
 			(effects (font (size 1.27 1.27)) (hide yes))
@@
 			(effects (font (size 1.27 1.27)))
 		)
-		(property "Footprint" "Resistor_SMD:R_0402_1005Metric"
+		(property "Footprint" "0402"
 			(at 203.2 50.8 0)
 			(effects (font (size 1.27 1.27)) (hide yes))
@@
 			(at 203.2 50.8 0)
 			(effects (font (size 1.27 1.27)) (hide yes))
+		)
+		(property "LCSC" "C25744"
+			(at 203.2 50.8 0)
+			(effects (font (size 1.27 1.27)) (hide yes))
+		)
+		(property "MPN" "0402WGF1002TCE"
+			(at 203.2 50.8 0)
+			(effects (font (size 1.27 1.27)) (hide yes))
