File: hardware/kicad/elderly-companion-robot/camera_dock.kicad_sch (KiCad schematic)
At the start: 0 parts

Commit message: Phase 9-10: All 6 hierarchical sheets populated with components, labels, and power symbols
- Power_Supply: LM2596S-5 buck, AP2112K-3.3 LDO, AMS1117-ADJ (4V for SIM800L),
  TP4056 charger, caps, diodes, connectors, resistor dividers
- MCU_Core: ESP32-S3-WROOM-1, 8x decoupling caps, boot/EN resistors,
  hierarchical labels for all peripheral interfaces
- Motor_Driver: L298N, 8x flyback diodes, motor connectors, hierarchical labels
- Sensors: MPU-6050, SSD1306 OLED, 4x HC-SR04 connectors, voltage dividers,
  I2C pull-ups, hierarchical labels
- Audio: MAX98357A, INMP441 connector (6-pin), speaker connector, bypass caps,
  I2S hierarchical labels
- Camera_Dock: SIM800C, 2x servo connectors, IR TX/RX, dock contact,
  UART2/PWRKEY hierarchical labels
- Top-level schematic restored with 6 hierarchical sheet references
- ERC: 0 violations
- Quality gate: Schematic PASS

Co-Authored-By: Claude Opus 4.7 <noreply@anthropic.com>
Parts:
- added C34: 100uF, Capacitor_SMD:CP_Elec_6.3x7.7, symbol Device:C_Polarized
- added C35: 100nF, Capacitor_SMD:C_0402_1005Metric, symbol Device:C
- added J11: Servo_Pan, Connector_PinHeader_2.54mm:PinHeader_1x03_P2.54mm_Vertical, symbol Connector_Generic:Conn_01x03
- added J12: Servo_Tilt, Connector_PinHeader_2.54mm:PinHeader_1x03_P2.54mm_Vertical, symbol Connector_Generic:Conn_01x03
- added J13: IR_TX_LED, Connector_PinHeader_2.54mm:PinHeader_1x02_P2.54mm_Vertical, symbol Connector_Generic:Conn_01x02
- added J14: IR_RX, Connector_PinHeader_2.54mm:PinHeader_1x02_P2.54mm_Vertical, symbol Connector_Generic:Conn_01x02
- added J15: Dock_Contact, Connector_PinHeader_2.54mm:PinHeader_1x02_P2.54mm_Vertical, symbol Connector_Generic:Conn_01x02
- added R18: 220, Resistor_SMD:R_0402_1005Metric, symbol Device:R
- added U9: SIM800C, RF_GSM:SIMCom_SIM800C, symbol RF_GSM:SIM800C
Connections:
- new net: J11.1 (Pin_1), U9.14 (SIM_DET)
- new net: J11.3 (Pin_3), U9.24 (USB_VBUS)
- new net: U9.13 (GND), U9.19 (GND), U9.21 (GND), U9.27 (GND), U9.30 (GND), U9.31 (GND), U9.33 (GND), U9.36 (GND), U9.37 (GND), U9.8 (GND)
- new net: U9.34 (VBAT), U9.35 (VBAT)
Other:
- title: Camera_Dock -> (none)

Commit message: LCSC part binding + all 6 sheets wired, ERC clean
- LCSC codes bound for passive components (caps, resistors, diodes, LEDs)
- Power Supply: LM2596S-5, AP2112K, AMS1117, TP4056 wired with nets
- MCU Core: ESP32-S3-WROOM-1 + decoupling caps + hierarchical labels
- Motor Driver: L298N + flyback diodes + connectors + labels
- Sensors: MPU-6050, SSD1306, 4x HC-SR04 + voltage dividers
- Audio: MAX98357A, INMP441 connector, speaker + I2S labels
- Camera/Dock: SIM800C, servos, IR, dock contact + UART2 labels
- ERC: 0 violations, schematic quality gate PASS

Co-Authored-By: Claude Opus 4.7 <noreply@anthropic.com>
Parts:
- C35: footprint Capacitor_SMD:C_0402_1005Metric -> 0402; LCSC (none) -> C1525; MPN (none) -> CL05B104KO5NNNC
- R18: footprint Resistor_SMD:R_0402_1005Metric -> 0402; LCSC (none) -> C25091; MPN (none) -> 0402WGF2200TCE
Changed lines of the file:
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@@
 			(effects (font (size 1.27 1.27)))
 		)
-		(property "Footprint" "Capacitor_SMD:C_0402_1005Metric"
+		(property "Footprint" "0402"
 			(at 228.6 50.8 0)
 			(effects (font (size 1.27 1.27)) (hide yes))
 		)
 		(property "Datasheet" "~"
+			(at 228.6 50.8 0)
+			(effects (font (size 1.27 1.27)) (hide yes))
+		)
+		(property "LCSC" "C1525"
+			(at 228.6 50.8 0)
+			(effects (font (size 1.27 1.27)) (hide yes))
+		)
+		(property "MPN" "CL05B104KO5NNNC"
 			(at 228.6 50.8 0)
 			(effects (font (size 1.27 1.27)) (hide yes))
@@
 			(effects (font (size 1.27 1.27)))
 		)
-		(property "Footprint" "Resistor_SMD:R_0402_1005Metric"
+		(property "Footprint" "0402"
 			(at 254 50.8 0)
 			(effects (font (size 1.27 1.27)) (hide yes))
@@
 			(at 254 50.8 0)
 			(effects (font (size 1.27 1.27)) (hide yes))
+		)
+		(property "LCSC" "C25091"
+			(at 254 50.8 0)
+			(effects (font (size 1.27 1.27)) (hide yes))
+		)
+		(property "MPN" "0402WGF2200TCE"
+			(at 254 50.8 0)
+			(effects (font (size 1.27 1.27)) (hide yes))
