File: hardware/kicad/elderly-companion-robot/mcu_core.kicad_sch (KiCad schematic)
At the start: 0 parts

Commit message: Phase 9-10: All 6 hierarchical sheets populated with components, labels, and power symbols
- Power_Supply: LM2596S-5 buck, AP2112K-3.3 LDO, AMS1117-ADJ (4V for SIM800L),
  TP4056 charger, caps, diodes, connectors, resistor dividers
- MCU_Core: ESP32-S3-WROOM-1, 8x decoupling caps, boot/EN resistors,
  hierarchical labels for all peripheral interfaces
- Motor_Driver: L298N, 8x flyback diodes, motor connectors, hierarchical labels
- Sensors: MPU-6050, SSD1306 OLED, 4x HC-SR04 connectors, voltage dividers,
  I2C pull-ups, hierarchical labels
- Audio: MAX98357A, INMP441 connector (6-pin), speaker connector, bypass caps,
  I2S hierarchical labels
- Camera_Dock: SIM800C, 2x servo connectors, IR TX/RX, dock contact,
  UART2/PWRKEY hierarchical labels
- Top-level schematic restored with 6 hierarchical sheet references
- ERC: 0 violations
- Quality gate: Schematic PASS

Co-Authored-By: Claude Opus 4.7 <noreply@anthropic.com>
Parts:
- added C20, C21, C22, C23, C24, C25, C26, C28, C29: 100nF, Capacitor_SMD:C_0402_1005Metric, symbol Device:C
- added C27: 10uF, Capacitor_SMD:C_0805_2012Metric, symbol Device:C
- added R10, R11, R12: 10K, Resistor_SMD:R_0402_1005Metric, symbol Device:R
- added SW1: BOOT, Button_Switch_SMD:SW_Push_1P1T_NO_6x6mm_H6.3mm, symbol Switch:SW_Push
- added U10: ESP32-S3-WROOM-1, RF_Module:ESP32-S3-WROOM-1, symbol RF_Module:ESP32-S3-WROOM-1
Connections:
- new net: U10.1 (GND), U10.40 (GND), U10.41 (GND)
Other:
- title: MCU_Core -> (none)

Commit message: LCSC part binding + all 6 sheets wired, ERC clean
- LCSC codes bound for passive components (caps, resistors, diodes, LEDs)
- Power Supply: LM2596S-5, AP2112K, AMS1117, TP4056 wired with nets
- MCU Core: ESP32-S3-WROOM-1 + decoupling caps + hierarchical labels
- Motor Driver: L298N + flyback diodes + connectors + labels
- Sensors: MPU-6050, SSD1306, 4x HC-SR04 + voltage dividers
- Audio: MAX98357A, INMP441 connector, speaker + I2S labels
- Camera/Dock: SIM800C, servos, IR, dock contact + UART2 labels
- ERC: 0 violations, schematic quality gate PASS

Co-Authored-By: Claude Opus 4.7 <noreply@anthropic.com>
Parts:
- C20, C21, C22, C23, C24, C25, C26, C28: footprint Capacitor_SMD:C_0402_1005Metric -> 0402; LCSC (none) -> C1525; MPN (none) -> CL05B104KO5NNNC
- C27: footprint Capacitor_SMD:C_0805_2012Metric -> 0805; LCSC (none) -> C15850; MPN (none) -> CL21A106KAYNNNE
- R10, R11, R12: footprint Resistor_SMD:R_0402_1005Metric -> 0402; LCSC (none) -> C25744; MPN (none) -> 0402WGF1002TCE
Changed lines of the file:
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@@
 			(effects (font (size 1.27 1.27)))
 		)
-		(property "Footprint" "Capacitor_SMD:C_0402_1005Metric"
+		(property "Footprint" "0402"
 			(at 76.2 50.8 0)
 			(effects (font (size 1.27 1.27)) (hide yes))
 		)
 		(property "Datasheet" "~"
+			(at 76.2 50.8 0)
+			(effects (font (size 1.27 1.27)) (hide yes))
+		)
+		(property "LCSC" "C1525"
+			(at 76.2 50.8 0)
+			(effects (font (size 1.27 1.27)) (hide yes))
+		)
+		(property "MPN" "CL05B104KO5NNNC"
 			(at 76.2 50.8 0)
 			(effects (font (size 1.27 1.27)) (hide yes))
@@
 			(effects (font (size 1.27 1.27)))
 		)
-		(property "Footprint" "Capacitor_SMD:C_0402_1005Metric"
+		(property "Footprint" "0402"
 			(at 101.6 50.8 0)
 			(effects (font (size 1.27 1.27)) (hide yes))
 		)
 		(property "Datasheet" "~"
+			(at 101.6 50.8 0)
+			(effects (font (size 1.27 1.27)) (hide yes))
+		)
+		(property "LCSC" "C1525"
+			(at 101.6 50.8 0)
+			(effects (font (size 1.27 1.27)) (hide yes))
+		)
+		(property "MPN" "CL05B104KO5NNNC"
 			(at 101.6 50.8 0)
 			(effects (font (size 1.27 1.27)) (hide yes))
@@
 			(effects (font (size 1.27 1.27)))
 		)
-		(property "Footprint" "Capacitor_SMD:C_0402_1005Metric"
+		(property "Footprint" "0402"
 			(at 127 50.8 0)
 			(effects (font (size 1.27 1.27)) (hide yes))
 		)
 		(property "Datasheet" "~"
+			(at 127 50.8 0)
+			(effects (font (size 1.27 1.27)) (hide yes))
+		)
+		(property "LCSC" "C1525"
+			(at 127 50.8 0)
+			(effects (font (size 1.27 1.27)) (hide yes))
+		)
+		(property "MPN" "CL05B104KO5NNNC"
 			(at 127 50.8 0)
 			(effects (font (size 1.27 1.27)) (hide yes))
@@
 			(effects (font (size 1.27 1.27)))
 		)
-		(property "Footprint" "Capacitor_SMD:C_0402_1005Metric"
+		(property "Footprint" "0402"
 			(at 152.4 50.8 0)
 			(effects (font (size 1.27 1.27)) (hide yes))
 		)
 		(property "Datasheet" "~"
+			(at 152.4 50.8 0)
+			(effects (font (size 1.27 1.27)) (hide yes))
+		)
+		(property "LCSC" "C1525"
+			(at 152.4 50.8 0)
+			(effects (font (size 1.27 1.27)) (hide yes))
+		)
+		(property "MPN" "CL05B104KO5NNNC"
 			(at 152.4 50.8 0)
 			(effects (font (size 1.27 1.27)) (hide yes))
@@
 			(effects (font (size 1.27 1.27)))
 		)
-		(property "Footprint" "Capacitor_SMD:C_0402_1005Metric"
+		(property "Footprint" "0402"
 			(at 177.8 50.8 0)
 			(effects (font (size 1.27 1.27)) (hide yes))
 		)
 		(property "Datasheet" "~"
+			(at 177.8 50.8 0)
+			(effects (font (size 1.27 1.27)) (hide yes))
+		)
+		(property "LCSC" "C1525"
+			(at 177.8 50.8 0)
+			(effects (font (size 1.27 1.27)) (hide yes))
+		)
+		(property "MPN" "CL05B104KO5NNNC"
 			(at 177.8 50.8 0)
 			(effects (font (size 1.27 1.27)) (hide yes))
@@
 			(effects (font (size 1.27 1.27)))
 		)
-		(property "Footprint" "Capacitor_SMD:C_0402_1005Metric"
+		(property "Footprint" "0402"
 			(at 203.2 50.8 0)
 			(effects (font (size 1.27 1.27)) (hide yes))
 		)
 		(property "Datasheet" "~"
+			(at 203.2 50.8 0)
+			(effects (font (size 1.27 1.27)) (hide yes))
+		)
+		(property "LCSC" "C1525"
+			(at 203.2 50.8 0)
+			(effects (font (size 1.27 1.27)) (hide yes))
+		)
+		(property "MPN" "CL05B104KO5NNNC"
 			(at 203.2 50.8 0)
 			(effects (font (size 1.27 1.27)) (hide yes))
@@
 			(effects (font (size 1.27 1.27)))
 		)
-		(property "Footprint" "Capacitor_SMD:C_0402_1005Metric"
+		(property "Footprint" "0402"
 			(at 228.6 50.8 0)
 			(effects (font (size 1.27 1.27)) (hide yes))
 		)
 		(property "Datasheet" "~"
+			(at 228.6 50.8 0)
+			(effects (font (size 1.27 1.27)) (hide yes))
+		)
+		(property "LCSC" "C1525"
+			(at 228.6 50.8 0)
+			(effects (font (size 1.27 1.27)) (hide yes))
+		)
+		(property "MPN" "CL05B104KO5NNNC"
 			(at 228.6 50.8 0)
 			(effects (font (size 1.27 1.27)) (hide yes))
@@
 			(effects (font (size 1.27 1.27)))
 		)
-		(property "Footprint" "Capacitor_SMD:C_0805_2012Metric"
+		(property "Footprint" "0805"
 			(at 254 50.8 0)
 			(effects (font (size 1.27 1.27)) (hide yes))
 		)
 		(property "Datasheet" "~"
+			(at 254 50.8 0)
+			(effects (font (size 1.27 1.27)) (hide yes))
+		)
+		(property "LCSC" "C15850"
+			(at 254 50.8 0)
+			(effects (font (size 1.27 1.27)) (hide yes))
+		)
+		(property "MPN" "CL21A106KAYNNNE"
 			(at 254 50.8 0)
 			(effects (font (size 1.27 1.27)) (hide yes))
@@
 			(effects (font (size 1.27 1.27)))
 		)
-		(property "Footprint" "Capacitor_SMD:C_0402_1005Metric"
+		(property "Footprint" "0402"
 			(at 50.8 68.58 0)
 			(effects (font (size 1.27 1.27)) (hide yes))
 		)
 		(property "Datasheet" "~"
+			(at 50.8 68.58 0)
+			(effects (font (size 1.27 1.27)) (hide yes))
+		)
+		(property "LCSC" "C1525"
+			(at 50.8 68.58 0)
+			(effects (font (size 1.27 1.27)) (hide yes))
+		)
+		(property "MPN" "CL05B104KO5NNNC"
 			(at 50.8 68.58 0)
 			(effects (font (size 1.27 1.27)) (hide yes))
@@
 			(effects (font (size 1.27 1.27)))
 		)
-		(property "Footprint" "Resistor_SMD:R_0402_1005Metric"
+		(property "Footprint" "0402"
 			(at 76.2 68.58 0)
 			(effects (font (size 1.27 1.27)) (hide yes))
 		)
 		(property "Datasheet" "~"
+			(at 76.2 68.58 0)
+			(effects (font (size 1.27 1.27)) (hide yes))
+		)
+		(property "LCSC" "C25744"
+			(at 76.2 68.58 0)
+			(effects (font (size 1.27 1.27)) (hide yes))
+		)
+		(property "MPN" "0402WGF1002TCE"
 			(at 76.2 68.58 0)
 			(effects (font (size 1.27 1.27)) (hide yes))
@@
 			(effects (font (size 1.27 1.27)))
 		)
-		(property "Footprint" "Resistor_SMD:R_0402_1005Metric"
+		(property "Footprint" "0402"
 			(at 101.6 68.58 0)
 			(effects (font (size 1.27 1.27)) (hide yes))
 		)
 		(property "Datasheet" "~"
+			(at 101.6 68.58 0)
+			(effects (font (size 1.27 1.27)) (hide yes))
+		)
+		(property "LCSC" "C25744"
+			(at 101.6 68.58 0)
+			(effects (font (size 1.27 1.27)) (hide yes))
+		)
+		(property "MPN" "0402WGF1002TCE"
 			(at 101.6 68.58 0)
 			(effects (font (size 1.27 1.27)) (hide yes))
@@
 			(effects (font (size 1.27 1.27)))
 		)
-		(property "Footprint" "Resistor_SMD:R_0402_1005Metric"
+		(property "Footprint" "0402"
 			(at 127 68.58 0)
 			(effects (font (size 1.27 1.27)) (hide yes))
@@
 			(at 127 68.58 0)
 			(effects (font (size 1.27 1.27)) (hide yes))
+		)
+		(property "LCSC" "C25744"
+			(at 127 68.58 0)
+			(effects (font (size 1.27 1.27)) (hide yes))
+		)
+		(property "MPN" "0402WGF1002TCE"
+			(at 127 68.58 0)
+			(effects (font (size 1.27 1.27)) (hide yes))
