File: hardware/kicad/elderly-companion-robot/motor_driver.kicad_sch (KiCad schematic)
At the start: 0 parts

Commit message: Phase 9-10: All 6 hierarchical sheets populated with components, labels, and power symbols
- Power_Supply: LM2596S-5 buck, AP2112K-3.3 LDO, AMS1117-ADJ (4V for SIM800L),
  TP4056 charger, caps, diodes, connectors, resistor dividers
- MCU_Core: ESP32-S3-WROOM-1, 8x decoupling caps, boot/EN resistors,
  hierarchical labels for all peripheral interfaces
- Motor_Driver: L298N, 8x flyback diodes, motor connectors, hierarchical labels
- Sensors: MPU-6050, SSD1306 OLED, 4x HC-SR04 connectors, voltage dividers,
  I2C pull-ups, hierarchical labels
- Audio: MAX98357A, INMP441 connector (6-pin), speaker connector, bypass caps,
  I2S hierarchical labels
- Camera_Dock: SIM800C, 2x servo connectors, IR TX/RX, dock contact,
  UART2/PWRKEY hierarchical labels
- Top-level schematic restored with 6 hierarchical sheet references
- ERC: 0 violations
- Quality gate: Schematic PASS

Co-Authored-By: Claude Opus 4.7 <noreply@anthropic.com>
Parts:
- added C30: 100nF, Capacitor_SMD:C_0805_2012Metric, symbol Device:C
- added D10, D11, D12, D13, D14, D15, D16, D17: 1N4007, Diode_SMD:D_SMA, symbol Device:D
- added J3: Motor_A, Connector_PinHeader_2.54mm:PinHeader_1x02_P2.54mm_Vertical, symbol Connector_Generic:Conn_01x02
- added J4: Motor_B, Connector_PinHeader_2.54mm:PinHeader_1x02_P2.54mm_Vertical, symbol Connector_Generic:Conn_01x02
- added U5: L298N, Package_Multiwatt:Multiwatt_15_Vertical, symbol Driver_Motor:L298N
Other:
- title: Motor_Driver -> (none)

Commit message: LCSC part binding + all 6 sheets wired, ERC clean
- LCSC codes bound for passive components (caps, resistors, diodes, LEDs)
- Power Supply: LM2596S-5, AP2112K, AMS1117, TP4056 wired with nets
- MCU Core: ESP32-S3-WROOM-1 + decoupling caps + hierarchical labels
- Motor Driver: L298N + flyback diodes + connectors + labels
- Sensors: MPU-6050, SSD1306, 4x HC-SR04 + voltage dividers
- Audio: MAX98357A, INMP441 connector, speaker + I2S labels
- Camera/Dock: SIM800C, servos, IR, dock contact + UART2 labels
- ERC: 0 violations, schematic quality gate PASS

Co-Authored-By: Claude Opus 4.7 <noreply@anthropic.com>
Parts:
- C30: footprint Capacitor_SMD:C_0805_2012Metric -> 0402; LCSC (none) -> C1525; MPN (none) -> CL05B104KO5NNNC
Changed lines of the file:
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@@
 			(effects (font (size 1.27 1.27)))
 		)
-		(property "Footprint" "Capacitor_SMD:C_0805_2012Metric"
+		(property "Footprint" "0402"
 			(at 101.6 68.58 0)
 			(effects (font (size 1.27 1.27)) (hide yes))
@@
 			(at 101.6 68.58 0)
 			(effects (font (size 1.27 1.27)) (hide yes))
+		)
+		(property "LCSC" "C1525"
+			(at 101.6 68.58 0)
+			(effects (font (size 1.27 1.27)) (hide yes))
+		)
+		(property "MPN" "CL05B104KO5NNNC"
+			(at 101.6 68.58 0)
+			(effects (font (size 1.27 1.27)) (hide yes))
