File: hardware/kicad/elderly-companion-robot/sensors.kicad_sch (KiCad schematic)
At the start: 0 parts

Commit message: Phase 9-10: All 6 hierarchical sheets populated with components, labels, and power symbols
- Power_Supply: LM2596S-5 buck, AP2112K-3.3 LDO, AMS1117-ADJ (4V for SIM800L),
  TP4056 charger, caps, diodes, connectors, resistor dividers
- MCU_Core: ESP32-S3-WROOM-1, 8x decoupling caps, boot/EN resistors,
  hierarchical labels for all peripheral interfaces
- Motor_Driver: L298N, 8x flyback diodes, motor connectors, hierarchical labels
- Sensors: MPU-6050, SSD1306 OLED, 4x HC-SR04 connectors, voltage dividers,
  I2C pull-ups, hierarchical labels
- Audio: MAX98357A, INMP441 connector (6-pin), speaker connector, bypass caps,
  I2S hierarchical labels
- Camera_Dock: SIM800C, 2x servo connectors, IR TX/RX, dock contact,
  UART2/PWRKEY hierarchical labels
- Top-level schematic restored with 6 hierarchical sheet references
- ERC: 0 violations
- Quality gate: Schematic PASS

Co-Authored-By: Claude Opus 4.7 <noreply@anthropic.com>
Parts:
- added J5: US_Front, Connector_PinHeader_2.54mm:PinHeader_1x04_P2.54mm_Vertical, symbol Connector_Generic:Conn_01x04
- added J6: US_Back, Connector_PinHeader_2.54mm:PinHeader_1x04_P2.54mm_Vertical, symbol Connector_Generic:Conn_01x04
- added J7: US_Left, Connector_PinHeader_2.54mm:PinHeader_1x04_P2.54mm_Vertical, symbol Connector_Generic:Conn_01x04
- added J8: US_Right, Connector_PinHeader_2.54mm:PinHeader_1x04_P2.54mm_Vertical, symbol Connector_Generic:Conn_01x04
- added R13, R14: 4.7K, Resistor_SMD:R_0402_1005Metric, symbol Device:R
- added R15: 1K, Resistor_SMD:R_0402_1005Metric, symbol Device:R
- added R16: 2K, Resistor_SMD:R_0402_1005Metric, symbol Device:R
- added U6: MPU-6050, Sensor_Motion:QFN-24-1EP_4x4mm_P0.5mm_EP2.7x2.7mm, symbol Sensor_Motion:MPU-6050
- added U7: SSD1306_OLED, Display_Graphic:ER_OLEDM0.91_1x-I2C, symbol Display_Graphic:ER_OLEDM0.91_1x-I2C
Other:
- title: Sensors -> (none)

Commit message: LCSC part binding + all 6 sheets wired, ERC clean
- LCSC codes bound for passive components (caps, resistors, diodes, LEDs)
- Power Supply: LM2596S-5, AP2112K, AMS1117, TP4056 wired with nets
- MCU Core: ESP32-S3-WROOM-1 + decoupling caps + hierarchical labels
- Motor Driver: L298N + flyback diodes + connectors + labels
- Sensors: MPU-6050, SSD1306, 4x HC-SR04 + voltage dividers
- Audio: MAX98357A, INMP441 connector, speaker + I2S labels
- Camera/Dock: SIM800C, servos, IR, dock contact + UART2 labels
- ERC: 0 violations, schematic quality gate PASS

Co-Authored-By: Claude Opus 4.7 <noreply@anthropic.com>
Parts:
- R13, R14: footprint Resistor_SMD:R_0402_1005Metric -> 0402; LCSC (none) -> C25900; MPN (none) -> 0402WGF4701TCE
- R15: footprint Resistor_SMD:R_0402_1005Metric -> 0402; LCSC (none) -> C11702; MPN (none) -> 0402WGF1001TCE
- R16: footprint Resistor_SMD:R_0402_1005Metric -> 0402; LCSC (none) -> C4109; MPN (none) -> 0402WGF2001TCE
Changed lines of the file:
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@@
 			(effects (font (size 1.27 1.27)))
 		)
-		(property "Footprint" "Resistor_SMD:R_0402_1005Metric"
+		(property "Footprint" "0402"
 			(at 101.6 50.8 0)
 			(effects (font (size 1.27 1.27)) (hide yes))
 		)
 		(property "Datasheet" "~"
+			(at 101.6 50.8 0)
+			(effects (font (size 1.27 1.27)) (hide yes))
+		)
+		(property "LCSC" "C25900"
+			(at 101.6 50.8 0)
+			(effects (font (size 1.27 1.27)) (hide yes))
+		)
+		(property "MPN" "0402WGF4701TCE"
 			(at 101.6 50.8 0)
 			(effects (font (size 1.27 1.27)) (hide yes))
@@
 			(effects (font (size 1.27 1.27)))
 		)
-		(property "Footprint" "Resistor_SMD:R_0402_1005Metric"
+		(property "Footprint" "0402"
 			(at 127 50.8 0)
 			(effects (font (size 1.27 1.27)) (hide yes))
 		)
 		(property "Datasheet" "~"
+			(at 127 50.8 0)
+			(effects (font (size 1.27 1.27)) (hide yes))
+		)
+		(property "LCSC" "C25900"
+			(at 127 50.8 0)
+			(effects (font (size 1.27 1.27)) (hide yes))
+		)
+		(property "MPN" "0402WGF4701TCE"
 			(at 127 50.8 0)
 			(effects (font (size 1.27 1.27)) (hide yes))
@@
 			(effects (font (size 1.27 1.27)))
 		)
-		(property "Footprint" "Resistor_SMD:R_0402_1005Metric"
+		(property "Footprint" "0402"
 			(at 152.4 50.8 0)
 			(effects (font (size 1.27 1.27)) (hide yes))
 		)
 		(property "Datasheet" "~"
+			(at 152.4 50.8 0)
+			(effects (font (size 1.27 1.27)) (hide yes))
+		)
+		(property "LCSC" "C11702"
+			(at 152.4 50.8 0)
+			(effects (font (size 1.27 1.27)) (hide yes))
+		)
+		(property "MPN" "0402WGF1001TCE"
 			(at 152.4 50.8 0)
 			(effects (font (size 1.27 1.27)) (hide yes))
@@
 			(effects (font (size 1.27 1.27)))
 		)
-		(property "Footprint" "Resistor_SMD:R_0402_1005Metric"
+		(property "Footprint" "0402"
 			(at 177.8 50.8 0)
 			(effects (font (size 1.27 1.27)) (hide yes))
@@
 			(at 177.8 50.8 0)
 			(effects (font (size 1.27 1.27)) (hide yes))
+		)
+		(property "LCSC" "C4109"
+			(at 177.8 50.8 0)
+			(effects (font (size 1.27 1.27)) (hide yes))
+		)
+		(property "MPN" "0402WGF2001TCE"
+			(at 177.8 50.8 0)
+			(effects (font (size 1.27 1.27)) (hide yes))
